Commit message: fixed lidar publisher configuration

File: urdf/wheelchair_model_lidar.urdf (robot description, URDF)
Before this commit: robot wheelchair_robot, 8 links, 7 joints
Joints:
- joint leftscan_joint: origin xyz=0.2 -0.35 0.15 rpy=0 0 0 -> xyz=0.2 -0.35 0.15 rpy=0.1 0.5 0
- joint rightscan_joint: origin xyz=-0.2 -0.35 0.15 rpy=-4 0 0 -> xyz=-0.2 -0.35 0.15 rpy=0.1 -0.5 0
