Commit message: Swapped left and right wheels for wheelchair model description

File: urdf/wheelchair_model.urdf (robot description, URDF)
Before this commit: robot wheelchair_robot, 3 links, 2 joints
Joints:
- joint left_wheel_joint: origin xyz=-0.25 -0.240 0 rpy=0 0 0 -> xyz=-0.25 0.240 0 rpy=0 0 0
- joint right_wheel_joint: origin xyz=-0.25 0.240 0 rpy=0 0 0 -> xyz=-0.25 -0.240 0 rpy=0 0 0

Commit message: Added castors to front of wheelchair URDF

File: urdf/wheelchair_model.urdf (robot description, URDF)
Before this commit: robot wheelchair_robot, 3 links, 2 joints
Links:
- added link left_castor, mass 1; collision cylinder length=0.06 radius=0.165; visual cylinder length=0.05 radius=0.1
- added link left_castor_link; visual box size=0.1 0.1 0.1
- added link right_castor, mass 1; collision cylinder length=0.06 radius=0.165; visual cylinder length=0.05 radius=0.1
- added link right_castor_link; visual box size=0.1 0.1 0.1
Joints:
- added joint left_castor_joint: type continuous, parent left_castor_link, child left_castor, origin xyz=0 0 -0.07 rpy=0 0 0, axis 0 1 0
- added joint left_castor_link_joint: type fixed, parent base_link, child left_castor_link, origin xyz=0.4 0.22 0
- added joint right_castor_joint: type continuous, parent right_castor_link, child right_castor, origin xyz=0 0 -0.07 rpy=0 0 0, axis 0 1 0
- added joint right_castor_link_joint: type fixed, parent base_link, child right_castor_link, origin xyz=0.4 -0.22 0

Commit message: fixed visual component of wheelchair_model.urdf

File: urdf/wheelchair_model.urdf (robot description, URDF)
Before this commit: robot wheelchair_robot, 8 links, 7 joints
Links:
- removed link base_link
- removed link left_castor
- removed link left_castor_link
- removed link left_wheel
- removed link right_castor
- removed link right_castor_link
- removed link right_wheel
- removed link world
- added link wheelchair_base_link, mass 1; collision box size=0.45 0.8 0.2; visual box size=0.45 0.8 0.2
- added link wheelchair_left_castor_link, mass 1; collision sphere radius=0.1; visual sphere radius=0.1
- added link wheelchair_left_wheel_link, mass 1; collision cylinder length=0.06 radius=0.165; visual cylinder length=0.06 radius=0.165
- added link wheelchair_right_castor_link, mass 1; collision sphere radius=0.1; visual sphere radius=0.1
- added link wheelchair_right_wheel_link, mass 1; collision cylinder length=0.06 radius=0.165; visual cylinder length=0.06 radius=0.165
Joints:
- removed joint fixed
- removed joint left_castor_joint
- removed joint left_castor_link_joint
- removed joint left_wheel_joint
- removed joint right_castor_joint
- removed joint right_castor_link_joint
- removed joint right_wheel_joint
- added joint wheelchair_base_link_left_castor_joint: type revolute, parent wheelchair_base_link, child wheelchair_left_castor_link, origin xyz=0.69882 0.88174 0.43379 rpy=0 0 0, axis 1 0 0, limit lower=-1.79769e+308 upper=1.79769e+308 effort=-1.0 velocity=-1.0
- added joint wheelchair_base_link_left_wheel_joint: type revolute, parent wheelchair_base_link, child wheelchair_left_wheel_link, origin xyz=0.2473  0.30924 0.5 rpy=0 0 0, axis 1 0 0, limit lower=-1.79769e+308 upper=1.79769e+308 effort=-1.0 velocity=-1.0
- added joint wheelchair_base_link_right_castor_joint: type revolute, parent wheelchair_base_link, child wheelchair_right_castor_link, origin xyz=0.30213 0.88032 0.43379 rpy=0 0 0, axis 1 0 0, limit lower=-1.79769e+308 upper=1.79769e+308 effort=-1.0 velocity=-1.0
- added joint wheelchair_base_link_right_wheel_joint: type revolute, parent wheelchair_base_link, child wheelchair_right_wheel_link, origin xyz=0.75965 0.30724 0.5 rpy=0 0 0, axis 1 0 0, limit lower=-1.79769e+308 upper=1.79769e+308 effort=-1.0 velocity=-1.0

Commit message: fixed typo and updated transform urdf

File: urdf/wheelchair_model.urdf (robot description, URDF)
Before this commit: robot wheelchair_robot, 5 links, 4 joints
Links:
- removed link wheelchair_base_link
- added link base_link, mass 1; collision box size=0.45 0.8 0.2; visual box size=0.45 0.8 0.2
Joints:
- joint wheelchair_base_link_left_castor_joint: parent wheelchair_base_link -> base_link
- joint wheelchair_base_link_left_wheel_joint: parent wheelchair_base_link -> base_link
- joint wheelchair_base_link_right_castor_joint: parent wheelchair_base_link -> base_link
- joint wheelchair_base_link_right_wheel_joint: parent wheelchair_base_link -> base_link

Commit message: changed to continuous joints!

File: urdf/wheelchair_model.urdf (robot description, URDF)
Before this commit: robot wheelchair_robot, 5 links, 4 joints
Joints:
- joint wheelchair_base_link_left_castor_joint: limit lower=-1.79769e+308 upper=1.79769e+308 effort=-1.0 velocity=-1.0 -> (none); type revolute -> continuous
- joint wheelchair_base_link_left_wheel_joint: limit lower=-1.79769e+308 upper=1.79769e+308 effort=-1.0 velocity=-1.0 -> (none); type revolute -> continuous
- joint wheelchair_base_link_right_castor_joint: limit lower=-1.79769e+308 upper=1.79769e+308 effort=-1.0 velocity=-1.0 -> (none); type revolute -> continuous
- joint wheelchair_base_link_right_wheel_joint: limit lower=-1.79769e+308 upper=1.79769e+308 effort=-1.0 velocity=-1.0 -> (none); type revolute -> continuous

Commit message: inverted x axis controls for urdf, using turtlebot diff drive

File: urdf/wheelchair_model.urdf (robot description, URDF)
Before this commit: robot wheelchair_robot, 5 links, 4 joints
Joints:
- joint wheelchair_base_link_left_wheel_joint: axis 1 0 0 -> -1 0 0
- joint wheelchair_base_link_right_wheel_joint: axis 1 0 0 -> -1 0 0

Commit message: changed mass and inertia - behaving much better

File: urdf/wheelchair_model.urdf (robot description, URDF)
Before this commit: robot wheelchair_robot, 5 links, 4 joints
Links:
- link base_link: mass 1 -> 10
- link wheelchair_left_wheel_link: mass 1 -> 10
- link wheelchair_right_wheel_link: mass 1 -> 10
Joints:
- joint wheelchair_base_link_left_castor_joint: origin xyz=0.69882 0.88174 0.43379 rpy=0 0 0 -> xyz=0.2 -0.4 -0.07 rpy=0 0 0; type continuous -> fixed
- joint wheelchair_base_link_left_wheel_joint: axis -1 0 0 -> 1 0 0; origin xyz=0.2473  0.30924 0.5 rpy=0 0 0 -> xyz=0.25  0.2 0 rpy=0 0 0
- joint wheelchair_base_link_right_castor_joint: origin xyz=0.30213 0.88032 0.43379 rpy=0 0 0 -> xyz=-0.2 -0.4 -0.07 rpy=0 0 0; type continuous -> fixed
- joint wheelchair_base_link_right_wheel_joint: axis -1 0 0 -> 1 0 0; origin xyz=0.75965 0.30724 0.5 rpy=0 0 0 -> xyz=-0.25 0.2 0 rpy=0 0 0

Commit message: added base_footprint link and joint

File: urdf/wheelchair_model.urdf (robot description, URDF)
Before this commit: robot wheelchair_robot, 5 links, 4 joints
Links:
- added link base_footprint
Joints:
- added joint base_footprint_link: type fixed, parent base_footprint, child base_link, origin xyz=0 0 0 rpy=0 0 0

Commit message: updated mass values - reflecting shift in centre of gravity

File: urdf/wheelchair_model.urdf (robot description, URDF)
Before this commit: robot wheelchair_robot, 6 links, 5 joints
Links:
- link base_link: mass 10 -> 5
- link wheelchair_left_castor_link: mass 1 -> 0
- link wheelchair_left_wheel_link: mass 10 -> 20
- link wheelchair_right_castor_link: mass 1 -> 0
- link wheelchair_right_wheel_link: mass 10 -> 20

Commit message: rplidar facing correct direction

File: urdf/wheelchair_model.urdf (robot description, URDF)
Before this commit: robot wheelchair_robot, 6 links, 5 joints
Links:
- added link base_scan, mass 0.114; collision cylinder length=0.0315 radius=0.055; visual mesh filename=package://wheelchair_description/meshes/rplidar-a2m4-r1.stl scale=0.001 0.001 0.001
Joints:
- added joint scan_joint: type fixed, parent base_link, child base_scan, origin xyz=-0.032 0 0.172 rpy=4.7121 3.1414 4.7121

Commit message: gazebo - fixed collisions issue with lidar urdf

File: urdf/wheelchair_model.urdf (robot description, URDF)
Before this commit: robot wheelchair_robot, 7 links, 6 joints
Links:
- removed link base_scan
- added link front_scan; collision cylinder length=0.0315 radius=0.055; visual mesh filename=package://wheelchair_description/meshes/rplidar-a2m4-r1.stl scale=0.001 0.001 0.001
Joints:
- joint scan_joint: child base_scan -> front_scan; origin xyz=-0.032 0 0.172 rpy=4.7121 3.1414 4.7121 -> xyz=0 -0.35 0.1 rpy=4.7121 3.1414 4.7121

Commit message: fixed visual centering of rplidar

File: urdf/wheelchair_model.urdf (robot description, URDF)
Before this commit: robot wheelchair_robot, 7 links, 6 joints
Joints:
- joint scan_joint: origin xyz=0 -0.35 0.1 rpy=4.7121 3.1414 4.7121 -> xyz=0 -0.35 0.15 rpy=0 0 0

Commit message: updated lidar range on wheelchair model

File: urdf/wheelchair_model.urdf (robot description, URDF)
Before this commit: robot wheelchair_robot, 7 links, 6 joints
Links:
- removed link front_scan
- added link laser; collision cylinder length=0.0315 radius=0.055; visual mesh filename=package://wheelchair_description/meshes/rplidar-a2m4-r1.stl scale=0.001 0.001 0.001
Joints:
- joint scan_joint: child front_scan -> laser

Commit message: added camera to urdf

File: urdf/wheelchair_model.urdf (robot description, URDF)
Before this commit: robot wheelchair_robot, 7 links, 6 joints
Links:
- added link zed_camera_center; visual mesh filename=package://wheelchair_description/meshes/ZED.stl
- added link zed_left_camera_frame
- added link zed_left_camera_optical_frame
- added link zed_right_camera_frame
- added link zed_right_camera_optical_frame
Joints:
- added joint zed_camera_center_joint: type fixed, parent base_footprint, child zed_camera_center, origin xyz=0 0 0 rpy=0 0 0
- added joint zed_left_camera_joint: type fixed, parent zed_camera_center, child zed_left_camera_frame, origin xyz=0 0.06 0 rpy=0 0 0
- added joint zed_left_camera_optical_joint: type fixed, parent zed_left_camera_frame, child zed_left_camera_optical_frame, origin xyz=0 0 0 rpy=-1.57079632679 0.0 -1.57079632679
- added joint zed_right_camera_joint: type fixed, parent zed_camera_center, child zed_right_camera_frame, origin xyz=0 -0.06 0 rpy=0 0 0
- added joint zed_right_camera_optical_joint: type fixed, parent zed_right_camera_frame, child zed_right_camera_optical_frame, origin xyz=0 0 0 rpy=-1.57079632679 0.0 -1.57079632679

Commit message: added zed camera to urdf

File: urdf/wheelchair_model.urdf (robot description, URDF)
Before this commit: robot wheelchair_robot, 12 links, 11 joints
Joints:
- joint zed_camera_center_joint: parent base_footprint -> base_link

Commit message: added limits to wheels and removed camera

File: urdf/wheelchair_model.urdf (robot description, URDF)
Before this commit: robot wheelchair_robot, 12 links, 11 joints
Links:
- removed link zed_camera_center
- removed link zed_left_camera_frame
- removed link zed_left_camera_optical_frame
- removed link zed_right_camera_frame
- removed link zed_right_camera_optical_frame
Joints:
- removed joint zed_camera_center_joint
- removed joint zed_left_camera_joint
- removed joint zed_left_camera_optical_joint
- removed joint zed_right_camera_joint
- removed joint zed_right_camera_optical_joint
- joint wheelchair_base_link_left_wheel_joint: limit (none) -> effort=100 velocity=100
- joint wheelchair_base_link_right_wheel_joint: limit (none) -> effort=100 velocity=100

Commit message: added camera to wheelchair model

File: urdf/wheelchair_model.urdf (robot description, URDF)
Before this commit: robot wheelchair_robot, 7 links, 6 joints
Links:
- added link zed_camera_center; visual mesh filename=package://wheelchair_description/meshes/ZED.stl
- added link zed_left_camera_frame
- added link zed_left_camera_optical_frame
- added link zed_right_camera_frame
- added link zed_right_camera_optical_frame
Joints:
- added joint zed_camera_center_joint: type fixed, parent base_link, child zed_camera_center, origin xyz=0 0 0 rpy=0 0 0
- added joint zed_left_camera_joint: type fixed, parent zed_camera_center, child zed_left_camera_frame, origin xyz=0 0.06 0 rpy=0 0 0
- added joint zed_left_camera_optical_joint: type fixed, parent zed_left_camera_frame, child zed_left_camera_optical_frame, origin xyz=0 0 0 rpy=-1.57079632679 0.0 -1.57079632679
- added joint zed_right_camera_joint: type fixed, parent zed_camera_center, child zed_right_camera_frame, origin xyz=0 -0.06 0 rpy=0 0 0
- added joint zed_right_camera_optical_joint: type fixed, parent zed_right_camera_frame, child zed_right_camera_optical_frame, origin xyz=0 0 0 rpy=-1.57079632679 0.0 -1.57079632679
