Commit message: imu working in urdf

File: urdf/wheelchair_model_fixing.urdf (robot description, URDF)
Before this commit: robot wheelchair_robot, 12 links, 11 joints
Links:
- added link imu; collision box size=0.03 0.02 0.01; visual box size=0.03 0.02 0.01
Joints:
- added joint imu_joint: type fixed, parent base_link, child imu, origin xyz=0 0 0.105, axis 1 0 0

Commit message: fixed viewing angle from parent camera link

File: urdf/wheelchair_model_fixing.urdf (robot description, URDF)
Before this commit: robot wheelchair_robot, 13 links, 12 joints
Joints:
- joint zed_camera_center_joint: origin xyz=0 0 0 rpy=0 0 0 -> xyz=0 0 0.45 rpy=0 0 0
