Commit message: updated world

File: urdf/wheelchair_model_tof7.urdf (robot description, URDF)
Before this commit: robot wheelchair_robot, 15 links, 14 joints
Links:
- added link zed_left_camera_stereo_frame
Joints:
- added joint zed_left_camera_stereo_joint: type fixed, parent zed_left_camera_frame, child zed_left_camera_stereo_frame, origin xyz=0 0 0 rpy=0 0 0

Commit message: fixing kinect zed axis

File: urdf/wheelchair_model_tof7.urdf (robot description, URDF)
Before this commit: robot wheelchair_robot, 16 links, 15 joints
Links:
- removed link zed_left_camera_stereo_frame
- added link zed_left_camera_depth_link
Joints:
- removed joint zed_left_camera_stereo_joint
- added joint zed_left_camera_depth_joint: type fixed, parent zed_left_camera_frame, child zed_left_camera_depth_link, origin xyz=0 0 0 rpy=0 0 0

Commit message: corrected base_link height

File: urdf/wheelchair_model_tof7.urdf (robot description, URDF)
Before this commit: robot wheelchair_robot, 16 links, 15 joints
Joints:
- joint base_footprint_link: origin xyz=0 0 0 rpy=0 0 0 -> xyz=0 0 0.17 rpy=0 0 0

Commit message: changed angle of camera - urdf

File: urdf/wheelchair_model_tof7.urdf (robot description, URDF)
Before this commit: robot wheelchair_robot, 16 links, 15 joints
Joints:
- joint zed_camera_center_joint: origin xyz=0 0 1.45 rpy=0 0 0 -> xyz=0 0 1.45 rpy=0 0.174533 0

Commit message: changed to 13 degree angle

File: urdf/wheelchair_model_tof7.urdf (robot description, URDF)
Before this commit: robot wheelchair_robot, 16 links, 15 joints
Joints:
- joint zed_camera_center_joint: origin xyz=0 0 1.45 rpy=0 0.174533 0 -> xyz=0 0 1.45 rpy=0 0.226893 0

Commit message: added height to camera

File: urdf/wheelchair_model_tof7.urdf (robot description, URDF)
Before this commit: robot wheelchair_robot, 16 links, 15 joints
Joints:
- joint zed_camera_center_joint: origin xyz=0 0 1.45 rpy=0 0.226893 0 -> xyz=0 0 1.55 rpy=0 0.226893 0

Commit message: raised height of robot

File: urdf/wheelchair_model_tof7.urdf (robot description, URDF)
Before this commit: robot wheelchair_robot, 16 links, 15 joints
Joints:
- joint base_footprint_link: origin xyz=0 0 0.17 rpy=0 0 0 -> xyz=0 0 0.25 rpy=0 0 0

Commit message: lowered camera height

File: urdf/wheelchair_model_tof7.urdf (robot description, URDF)
Before this commit: robot wheelchair_robot, 16 links, 15 joints
Joints:
- joint zed_camera_center_joint: origin xyz=0 0 1.55 rpy=0 0.226893 0 -> xyz=0 0 1.45 rpy=0 0.226893 0

Commit message: lowered camera height

File: urdf/wheelchair_model_tof7.urdf (robot description, URDF)
Before this commit: robot wheelchair_robot, 16 links, 15 joints
Joints:
- joint zed_camera_center_joint: origin xyz=0 0 1.45 rpy=0 0.226893 0 -> xyz=0 0 1.35 rpy=0 0.226893 0

Commit message: lowered camera height

File: urdf/wheelchair_model_tof7.urdf (robot description, URDF)
Before this commit: robot wheelchair_robot, 16 links, 15 joints
Joints:
- joint zed_camera_center_joint: origin xyz=0 0 1.35 rpy=0 0.226893 0 -> xyz=0 0 1.25 rpy=0 0.226893 0

Commit message: lowered camera height

File: urdf/wheelchair_model_tof7.urdf (robot description, URDF)
Before this commit: robot wheelchair_robot, 16 links, 15 joints
Joints:
- joint zed_camera_center_joint: origin xyz=0 0 1.25 rpy=0 0.226893 0 -> xyz=0 0 1.05 rpy=0 0.226893 0

Commit message: changed name of depth frame parent

File: urdf/wheelchair_model_tof7.urdf (robot description, URDF)
Before this commit: robot wheelchair_robot, 16 links, 15 joints
Joints:
- joint zed_left_camera_depth_joint: parent zed_left_camera_frame -> zed_left_camera_optical_frame

Commit message: added dummy base link inertia, renamed from base_footprint to base_link

File: urdf/wheelchair_model_tof7.urdf (robot description, URDF)
Before this commit: robot wheelchair_robot, 16 links, 15 joints
Links:
- removed link base_footprint
- added link base_link_dummy, mass 5; collision box size=0.72 0.51 0.25; visual box size=0.72 0.51 0.25
- link base_link: mass 5 -> None; geometry 
Joints:
- removed joint base_footprint_link
- added joint base_link_dummy_link: type fixed, parent base_link, child base_link_dummy, origin xyz=0 0 0.25 rpy=0 0 0

Commit message: moved joints further up from base_link

File: urdf/wheelchair_model_tof7.urdf (robot description, URDF)
Before this commit: robot wheelchair_robot, 16 links, 15 joints
Joints:
- joint deck1_joint: origin xyz=0 0 0.25 rpy=0 0 0 -> xyz=0 0 0.5 rpy=0 0 0
- joint deck2_joint: origin xyz=0 0 0.35 rpy=0 0 0 -> xyz=0 0 0.6 rpy=0 0 0
- joint wheelchair_base_link_left_castor_joint: origin xyz=0.4 0.16 -0.1 rpy=0 0 0 -> xyz=0.4 0.16 0.15 rpy=0 0 0
- joint wheelchair_base_link_left_wheel_joint: origin xyz=-0.2  0.23 -0.05 rpy=0 0 0 -> xyz=-0.2  0.23 0.2 rpy=0 0 0
- joint wheelchair_base_link_right_castor_joint: origin xyz=0.4 -0.16 -0.1 rpy=0 0 0 -> xyz=0.4 -0.16 0.15 rpy=0 0 0
- joint wheelchair_base_link_right_wheel_joint: origin xyz=-0.2 -0.23 -0.05 rpy=0 0 0 -> xyz=-0.2 -0.23 0.2 rpy=0 0 0
- joint zed_camera_center_joint: origin xyz=0 0 1.05 rpy=0 0.226893 0 -> xyz=0 0 1.3 rpy=0 0.226893 0

Commit message: updated height of laser

File: urdf/wheelchair_model_tof7.urdf (robot description, URDF)
Before this commit: robot wheelchair_robot, 16 links, 15 joints
Joints:
- joint scan_joint: origin xyz=0.35 0 0.15 rpy=0 0 0 -> xyz=0.35 0 0.4 rpy=0 0 0
